Commit message: Fixed controller

File: config/motoman_sia5f.ros2_control.xacro (robot description, xacro)
@@ -2,5 +2,5 @@
 <robot xmlns:xacro="http://www.ros.org/wiki/xacro">
     <xacro:macro name="motoman_sia5f_ros2_control" params="name initial_positions_file">
-        <xacro:property name="initial_positions" value="${load_yaml(initial_positions_file)['initial_positions']}"/>
+        <xacro:property name="initial_positions" value="${xacro.load_yaml(initial_positions_file)['initial_positions']}"/>
         <ros2_control name="${name}" type="system">
             <hardware>

Commit message: add demo with simulation parameter

File: config/motoman_sia5f.ros2_control.xacro (robot description, xacro)
@@ -57,8 +57,8 @@
                 <state_interface name="velocity"/>
             </joint>
-            <joint name="right_joint">
+            <joint name="gripper_joint">
                 <command_interface name="position"/>
                 <state_interface name="position">
-                  <param name="initial_value">${initial_positions['right_joint']}</param>
+                  <param name="initial_value">${initial_positions['gripper_joint']}</param>
                 </state_interface>
                 <state_interface name="velocity"/>

File: config/motoman_sia5f.urdf.xacro (robot description, xacro)
@@ -3,5 +3,5 @@
     <xacro:arg name="initial_positions_file" default="initial_positions.yaml" />
     <!-- Import motoman_sia5f urdf file -->
-    <xacro:include filename="$(find gazebo_simulation_ros2)/description/manipulator.urdf.xacro" />
+    <xacro:include filename="$(find uclv_yaskawa_simulation)/description/manipulator.urdf.xacro" />
     <!-- Import control_xacro -->
     <xacro:include filename="motoman_sia5f.ros2_control.xacro" />
